Commit message: correcting diffbot_controller params

File: description/urdf/diffbot_description.urdf.xacro (robot description, xacro)
@@ -2,27 +2,35 @@
 <robot xmlns:xacro="http://www.ros.org/wiki/xacro">
   <xacro:macro name="diffbot" params="prefix">
-  <!-- Constants for robot dimensions -->
-  <xacro:property name="base_width" value="0.1" />
-  <xacro:property name="base_height" value="0.05" />
-  <xacro:property name="z_offset" value="-${base_height/2}" /> <!-- Space btw top of beam and the each joint -->
-  <!-- Base Link -->
-  <link name="${prefix}base_link"></link>
-  <link name="${prefix}left_wheel"></link>
-  <link name="${prefix}right_wheel"></link>
+    <!-- Constants for robot dimensions -->
+    <xacro:property name="base_width" value="0.1" />
+    <xacro:property name="base_height" value="0.05" />
+    <xacro:property name="z_offset" value="-${base_height/2}" /> <!-- Space btw top of beam and the
+    each joint -->
+    <!-- Base Link -->
+    <link name="${prefix}base_link"></link>
+    <link name="${prefix}left_wheel"></link>
+    <link name="${prefix}right_wheel"></link>
+    <link name="${prefix}laser"></link>
+    <joint name="joint_rp" type="fixed">
+      <origin xyz="0.2 0.0 0.0" rpy="0.0 0 0.0" />
+      <parent link="${prefix}base_link" />
+      <child link="${prefix}laser" />
+      <axis xyz="0 0 0" />
+    </joint>
     <joint name="${prefix}left_wheel_joint" type="continuous">
-      <parent link="${prefix}base_link"/>
-      <child link="${prefix}left_wheel"/>
-      <origin xyz="0 -${base_width/2} ${z_offset}" rpy="0 0 0"/>
-      <axis xyz="0 1 0"/>
-      <dynamics damping="0.2"/>
-      <limit effort="100" velocity="1.0"/>
+      <parent link="${prefix}base_link" />
+      <child link="${prefix}left_wheel" />
+      <origin xyz="0 -${base_width/2} ${z_offset}" rpy="0 0 0" />
+      <axis xyz="0 1 0" />
+      <dynamics damping="0.2" />
+      <limit effort="100" velocity="1.0" />
     </joint>
     <joint name="${prefix}right_wheel_joint" type="continuous">
-      <parent link="${prefix}base_link"/>
-      <child link="${prefix}right_wheel"/>
-      <origin xyz="0 ${base_width/2} ${z_offset}" rpy="0 0 0"/>
-      <axis xyz="0 1 0"/>
-      <dynamics damping="0.2"/>
-      <limit effort="100" velocity="1.0"/>
+      <parent link="${prefix}base_link" />
+      <child link="${prefix}right_wheel" />
+      <origin xyz="0 ${base_width/2} ${z_offset}" rpy="0 0 0" />
+      <axis xyz="0 1 0" />
+      <dynamics damping="0.2" />
+      <limit effort="100" velocity="1.0" />
     </joint>
   </xacro:macro>
